Commit message: wheels are rotating in gazebo, however it is not moving around

File: src/intro_rover_description/urdf/intro_rover_description.urdf (robot description, URDF)
Before this commit: robot intro_rover_description, 15 links, 14 joints
Links:
- link base_link: geometry collision box size=0.60 0.45 0.20; visual mesh filename=package://intro_rover_description/meshes/base_link.STL
- link bl_swerve_yaw_link: mass 0.554469856268406 -> 0.55447
- link bl_wheel_link: mass 1.55830610436698 -> 1.5583; geometry collision cylinder length=0.08 radius=0.14; visual mesh filename=package://intro_rover_description/meshes/bl_wheel_link.STL
- link br_swerve_yaw_link: mass 0.554469856210505 -> 0.55447
- link br_wheel_link: mass 1.5583061724315 -> 1.5583; geometry collision cylinder length=0.08 radius=0.14; visual mesh filename=package://intro_rover_description/meshes/br_wheel_link.STL
- link fl_swerve_yaw_link: mass 0.554469856210505 -> 0.55447
- link fl_wheel_link: mass 1.55830614121036 -> 1.5583; geometry collision cylinder length=0.08 radius=0.14; visual mesh filename=package://intro_rover_description/meshes/fl_wheel_link.STL
- link fr_swerve_yaw_link: mass 0.554469856268406 -> 0.55447
- link fr_wheel_link: mass 1.55830616496123 -> 1.5583; geometry collision cylinder length=0.08 radius=0.14; visual mesh filename=package://intro_rover_description/meshes/fr_wheel_link.STL
Joints:
- joint bl_swerve_yaw: limit lower=-1.57 upper=1.57 effort=10 velocity=1 -> lower=-1.57 upper=1.57 effort=20.0 velocity=4.0; origin xyz=-0.466299868071487 0.514883785757828 -0.0484375000000003 rpy=0 0 0 -> xyz=-0.4662998 0.5148838 -0.0484375 rpy=0 0 0
- joint bl_wheel: axis 0 -1 0 -> 0 1 0; limit (none) -> effort=40.0 velocity=20.0; origin xyz=-0.000212360752061991 0.0574662142421849 -0.201583720606049 rpy=0 0 0 -> xyz=-0.0002124 0.0574662 -0.2015837 rpy=0 0 0
- joint br_swerve_yaw: limit lower=-1.57 upper=1.57 effort=10 velocity=1 -> lower=-1.57 upper=1.57 effort=20.0 velocity=4.0
- joint br_wheel: limit (none) -> effort=40.0 velocity=20.0; origin xyz=-0.00021041711699632 -0.0574662142420289 -0.201522792567001 rpy=0 0 0 -> xyz=-0.0002104 -0.0574662 -0.2015228 rpy=0 0 0
- joint elbow_pitch: limit lower=-1.57 upper=1.57 effort=10 velocity=1 -> lower=-1.57 upper=1.57 effort=30.0 velocity=2.0
- joint elbow_roll: limit (none) -> effort=15.0 velocity=3.0
- joint fl_swerve_yaw: limit lower=-1.57 upper=1.57 effort=10 velocity=1 -> lower=-1.57 upper=1.57 effort=20.0 velocity=4.0
- joint fl_wheel: axis 0 -1 0 -> 0 1 0; limit (none) -> effort=40.0 velocity=20.0; origin xyz=0.000210417116996542 0.0574662142421208 -0.201522792567001 rpy=0 0 0 -> xyz=0.0002104 0.0574662 -0.2015228 rpy=0 0 0
- joint fr_swerve_yaw: limit lower=-1.57 upper=1.57 effort=10 velocity=1 -> lower=-1.57 upper=1.57 effort=20.0 velocity=4.0
- joint fr_wheel: limit (none) -> effort=40.0 velocity=20.0; origin xyz=0.000212360752061935 -0.0574662142422728 -0.201583720606049 rpy=0 0 0 -> xyz=0.00021236 -0.0574662 -0.2015837 rpy=0 0 0
- joint shoulder_pitch: limit lower=-1.57 upper=1.57 effort=10 velocity=1 -> lower=-1.57 upper=1.57 effort=30.0 velocity=2.0
- joint shoulder_yaw: limit (none) -> effort=30.0 velocity=2.0
- joint wrist_pitch: limit lower=-1.57 upper=1.57 effort=10 velocity=1 -> lower=-1.57 upper=1.57 effort=15.0 velocity=3.0
- joint wrist_roll: limit (none) -> effort=10.0 velocity=3.0
